File: LINBoard-HW/LINBoard-HW.kicad_pcb (KiCad board)
At the start: 4 copper layers, 70 x 81 mm, 67 parts, among them J1 TC, J2 TYPE-C 16PLT-H10.0, J4 ATM15-6P-BM03, SW1 BOOT, SW2 RESET, U1 PCA82C250, U2 TJA1029T, U3 TPS56339DDC, U4 LD1117S33CTR, U6 STM32F302C8Tx, Y1 8mHz

Commit message: doing some layout
Parts:
- removed C15: 1uF, Capacitor_SMD:C_0402_1005Metric
- removed FB1: FerriteBead_Small, Resistor_SMD:R_0402_1005Metric
- C1, C10, C11, C2, C24, C25, C26, C27, C28, C29, C3, C30, C31, C4, C7, C8, C9: footprint Capacitor_SMD:C_0402_1005Metric -> Capacitor_SMD:C_0805_2012Metric
- C12: value 100nF -> 4.7uF; footprint Capacitor_SMD:C_0402_1005Metric -> Capacitor_SMD:C_0805_2012Metric
- C13: value 4.7uF -> 10nF; footprint Capacitor_SMD:C_0402_1005Metric -> Capacitor_SMD:C_0805_2012Metric
- C14: value 100nF -> 1uF; footprint Capacitor_SMD:C_0402_1005Metric -> Capacitor_SMD:C_0805_2012Metric
- D5, D6, D7, D8: footprint LED_SMD:LED_0603_1608Metric -> LED_SMD:LED_0805_2012Metric
- R1, R13, R14, R2, R21, R22, R23, R24, R3, R4, R5, R6, R7: footprint Resistor_SMD:R_0402_1005Metric -> Resistor_SMD:R_0805_2012Metric
- moved C31 76.3 mm to (25.0, 26.8), turned to 90 degrees
- moved JP5 70.4 mm to (30.8, 22.2), turned to 0 degrees
- moved R24 70.1 mm to (28.6, 22.2), turned to 90 degrees
- moved D6 69.9 mm to (26.2, 22.2), turned to 0 degrees
- moved C2 65.0 mm to (34.9, 17.6), turned to 180 degrees
- moved C1 62.5 mm to (35.7, 15.6), turned to 90 degrees
- moved D1 61.2 mm to (33.9, 15.1), turned to 90 degrees
- moved JP6 60.5 mm to (31.4, 15.1), turned to 90 degrees
- moved D2 59.7 mm to (28.6, 14.8), turned to -90 degrees
- moved R1 57.3 mm to (31.4, 12.8), turned to 0 degrees
- moved R23 55.1 mm to (28.8, 11.5), turned to 180 degrees
- moved R21 54.2 mm to (34.7, 9.83), turned to 0 degrees
- moved C27 54.1 mm to (36.4, 9.22), turned to 90 degrees
- moved R22 53.3 mm to (28.8, 10.2), turned to 0 degrees
- moved U3 51.7 mm to (31.7, 8.67), turned to -90 degrees
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Connections:
- JP1 pad 2: /Microcontroller/UART2_TX -> /LIN/TX
- JP2 pad 2: /Microcontroller/UART2_RX -> /LIN/RX
- U6 pad 9: Net-(U6-VDDA) -> +3V3
Routing:
- net GND: track 0.00 -> 30.4 mm, vias 0 -> 6
- net /Connectors/VBUS: track 0.00 -> 15.2 mm, vias 0 -> 3
- net Net-(U6-PA15): track 0.00 -> 12.9 mm, vias 0 -> 1
- net Net-(U6-PB7): track 0.00 -> 12.3 mm
- net /CAN/STANDBY: track 0.00 -> 11.5 mm
- net /CAN/RX: track 0.00 -> 10.1 mm
- net Net-(J2-CC2): track 0.00 -> 8.47 mm
- net Net-(U6-PF0): track 0.00 -> 8.03 mm
- net Net-(U6-PF1): track 0.00 -> 8.01 mm
- net /CAN/TX: track 0.00 -> 7.86 mm
- net /Microcontroller/NRST: track 0.00 -> 7.52 mm, vias 0 -> 1
- net +3V3: track 0.00 -> 7.36 mm, vias 0 -> 1
- net /Microcontroller/SWDIO: track 0.00 -> 7.30 mm
- net Net-(J2-CC1): track 0.00 -> 6.03 mm
- net /Connectors/USB_D-: track 0.00 -> 5.82 mm, vias 0 -> 1
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Other:
- board size 70 x 81 mm -> 45.4 x 56 mm

Commit message: routing first pass complete
Parts:
- removed D3: Schottky, Diode_SMD:D_SOD-123
- removed J2: TYPE-C 16PLT-H10.0, Connector_USB:USB_C_Receptacle_GCT_USB4085
- removed JP6: MASTER, Jumper:SolderJumper-2_P1.3mm_Bridged_RoundedPad1.0x1.5mm
- added C5: 100nF, Capacitor_SMD:C_0805_2012Metric, F.Cu at (11.8, 33.0)
- added D9: Schottky, Diode_SMD:D_SOD-123, F.Cu at (18.2, -5.60)
- added J3: USB_C_Receptacle_USB2.0, Connector_USB:USB_C_Receptacle_GCT_USB4085, F.Cu at (-1.95, 42.7)
- added R8: 10K, Resistor_SMD:R_0805_2012Metric, F.Cu at (14.8, 27.8)
- added R9: 10K, Resistor_SMD:R_0805_2012Metric, F.Cu at (18.4, 27.8)
- added SW3: MASTER, SlideSwitch:CJS-1200TB, F.Cu at (-15.0, 21.9)
- added U5: MB85RC256V, Package_SO:SOIC-8_3.9x4.9mm_P1.27mm, F.Cu at (16.9, 31.7)
- TP3: value E_I2C1_SCL -> SDA
- TP4: value E_I2C1_SDA -> SCL
- moved C30 71.2 mm to (16.7, 24.0), turned to -90 degrees
- moved C3 55.2 mm to (14.6, 24.0), turned to -90 degrees
- moved C2 54.0 mm to (-17.9, 28.8), turned to -90 degrees
- moved JP5 51.4 mm to (-17.6, 39.4), turned to 90 degrees
- moved R24 50.6 mm to (-17.6, 43.0), turned to -90 degrees
- moved D6 50.2 mm to (-17.6, 46.6), turned to 90 degrees
- moved R4 50.0 mm to (6.80, 24.6), turned to -90 degrees
- moved R1 48.7 mm to (-17.2, 16.8), turned to -90 degrees
- moved C14 48.5 mm to (-5.20, 25.4), turned to 90 degrees
- moved C10 47.7 mm to (5.20, 30.0)
- moved D2 45.8 mm to (-17.2, 12.4), turned to 90 degrees
- moved C12 44.1 mm to (7.80, 27.8)
- moved C13 43.5 mm to (-5.80, 28.4), turned to 180 degrees
- moved D1 39.2 mm to (-5.20, 18.2), turned to -90 degrees
- moved R2 39.1 mm to (-15.5, 28.7)
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Connections:
- C10 pad 1: +3V3 -> +3.3V
- C11 pad 1: +3V3 -> +3.3V
- C12 pad 1: +3V3 -> +3.3V
- C13 pad 1: +3V3 -> +3.3V
- C14 pad 1: +3V3 -> +3.3V
- C9 pad 1: +3V3 -> +3.3V
- D4 pad 1: CAN_H -> CAN_L
- D4 pad 2: CAN_L -> CAN_H
- J1 pad 1: +3V3 -> +3.3V
- J4 pad 1: +12V -> CAN_L
- J4 pad 2: LIN -> CAN_H
- J4 pad 3: CAN_L -> LIN
- J4 pad 4: CAN_H -> GND
- J4 pad 6: GND -> +12V
- R4 pad 1: +3V3 -> +3.3V
- SW1 pad 3: +3V3 -> +3.3V
- TP3 pad 1: Net-(U6-PA15) -> /Microcontroller/I2C1_SDA
- TP4 pad 1: Net-(U6-PB7) -> /Microcontroller/I2C1_SCL
- U1 pad 5: +3V3 -> +3.3V
- U6 pad 1: +3V3 -> +3.3V
- U6 pad 24: +3V3 -> +3.3V
- U6 pad 36: +3V3 -> +3.3V
- U6 pad 38: Net-(U6-PA15) -> /Microcontroller/I2C1_SCL
- U6 pad 43: Net-(U6-PB7) -> /Microcontroller/I2C1_SDA
- U6 pad 48: +3V3 -> +3.3V
- U6 pad 9: +3V3 -> +3.3V
Routing:
- net +12P: track 0.00 -> 66.2 mm
- net +5V: track 0.00 -> 60.5 mm
- net +3.3V: track 0.00 -> 54.3 mm, vias 0 -> 17
- net /Microcontroller/I2C1_SCL: track 0.00 -> 32.6 mm, vias 0 -> 2
- net /Microcontroller/I2C1_SDA: track 0.00 -> 26.1 mm, vias 0 -> 2
- net +12V: track 0.00 -> 22.2 mm
- net /Microcontroller/NRST: track 7.52 -> 28.2 mm, vias 1 -> 2
- net LIN: track 0.00 -> 20.0 mm
- net Net-(U3-FB): track 0.00 -> 18.3 mm
- net GND: track 30.4 -> 48.2 mm, vias 6 -> 33
- net CAN_H: track 0.00 -> 16.4 mm
- net CAN_L: track 0.00 -> 13.8 mm
- net Net-(U6-PA15): track 12.9 -> 0.00 mm, vias 1 -> 0
- net Net-(U6-PB0): track 0.00 -> 12.7 mm
- net Net-(U6-PB7): track 12.3 -> 0.00 mm
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- added copper zone on F.Cu, net +12P
- added copper zone on F.Cu, net +5V
- added copper zone on F.Cu, net /Power/SW
Other:
- board text added: "1"
- board text added: "2"
- board text added: "3"
- board text added: "BOOT"
- board text added: "LINBoard v1"
- board text added: "M"
- board text added: "RST"
- board text added: "RX"
- board text added: "S"
- board text added: "SCL"
- board text added: "SDA"
- board text added: "TX"

Commit message: clean up
Routing:
- net +12P: track 66.2 -> 77.9 mm
- net /Microcontroller/I2C1_SDA: track 26.1 -> 23.6 mm
- net /Microcontroller/I2C1_SCL: track 32.6 -> 30.0 mm
- net +3.3V: track 54.3 -> 56.8 mm, vias 17 -> 21
- net GND: vias 33 -> 39
Other:
- board size 45.4 x 56 mm -> 46 x 56 mm

Commit message: fixed some trace widths
Parts:
- added G1: DingoFace, DRTLogo:DingoFaceNoFill, B.Cu at (0.80, 27.3)
- added R10: 5.1K, Resistor_SMD:R_0805_2012Metric, F.Cu at (8.30, 42.5)
- moved J1 0.80 mm to (11.6, 39.4)
Routing:
- net /Connectors/USB_D+: track 5.82 -> 12.0 mm
- net GND: track 48.2 -> 44.0 mm, vias 39 -> 52
- net /LIN/RX: track 9.21 -> 7.33 mm
- net +3.3V: track 56.8 -> 58.3 mm, vias 21 -> 17
- net /Microcontroller/SWO: track 6.61 -> 7.41 mm
- net /Microcontroller/SWCLK: track 6.72 -> 7.52 mm
- net /Microcontroller/SWDIO: track 10.4 -> 11.2 mm
Other:
- board text added: "1-CAN L 2-CAN H 3-LIN 4-GND 5-GND 6-12V"
