File: LINBoard-HW/LIN.kicad_sch (KiCad schematic)
At the start: 8 parts, among them SW1 MASTER, U2 TJA1029T

Commit message: board layout started
Parts:
- removed SW1: MASTER, symbol Switch:SW_SPDT
- added JP6: MASTER, Jumper:SolderJumper-2_P1.3mm_Bridged_RoundedPad1.0x1.5mm, symbol Jumper:Jumper_2_Small_Bridged
- C1, C2: footprint Capacitor_SMD:C_0603_1608Metric -> Capacitor_SMD:C_0402_1005Metric
- D1: footprint (none) -> Diode_SMD:D_SOD-323
- D2: value D_Schottky_Small_Filled -> Schottky; footprint (none) -> Diode_SMD:D_SOD-123
- R1, R2: footprint Resistor_SMD:R_0603_1608Metric -> Resistor_SMD:R_0402_1005Metric
Connections:
- net +12P: no longer R2.1
- net LIN: now also JP6.1 (A)
- net at R1.2: now also JP6.2 (B)
- new net +3.3V: R2.1
- no-connect marks 1 -> 0
Other:
- moved on the sheet: D2, R1
Changed lines of the file:
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@@
-	)
-	(junction
-		(at 119.38 80.01)
-		(diameter 0)
-		(color 0 0 0 0)
 	)
 	(junction
@@
 		(color 0 0 0 0)
 	)
-	(no_connect
-		(at 161.29 95.25)
-	)
-	(wire
-		(pts
-			(xy 163.83 105.41) (xy 163.83 106.68)
+	(wire
+		(pts
+			(xy 163.83 102.87) (xy 163.83 106.68)
 		)
 		(stroke
@@
 	(wire
 		(pts
-			(xy 166.37 86.36) (xy 166.37 88.9)
+			(xy 163.83 86.36) (xy 163.83 88.9)
 		)
 		(stroke
@@
 	(wire
 		(pts
-			(xy 166.37 93.98) (xy 166.37 95.25)
+			(xy 111.76 87.63) (xy 111.76 90.17)
+		)
+		(stroke
+			(width 0)
+			(type default)
+		)
+	)
+	(wire
+		(pts
+			(xy 163.83 93.98) (xy 163.83 97.79)
 		)
 		(stroke
@@
 	(wire
 		(pts
-			(xy 111.76 80.01) (xy 119.38 80.01)
-		)
-		(stroke
-			(width 0)
-			(type default)
-		)
-	)
-	(wire
-		(pts
 			(xy 143.51 106.68) (xy 157.48 106.68)
 		)
@@
 	(wire
 		(pts
-			(xy 166.37 77.47) (xy 130.81 77.47)
-		)
-		(stroke
-			(width 0)
-			(type default)
-		)
-	)
-	(wire
-		(pts
-			(xy 111.76 90.17) (xy 111.76 80.01)
-		)
-		(stroke
-			(width 0)
-			(type default)
-		)
-	)
-	(wire
-		(pts
-			(xy 166.37 81.28) (xy 166.37 77.47)
+			(xy 163.83 77.47) (xy 130.81 77.47)
+		)
+		(stroke
+			(width 0)
+			(type default)
+		)
+	)
+	(wire
+		(pts
+			(xy 163.83 81.28) (xy 163.83 77.47)
 		)
 		(stroke
@@
 	)
 	(symbol
-		(lib_id "Switch:SW_SPDT")
+		(lib_id "Jumper:Jumper_2_Small_Bridged")
 		(at 163.83 100.33 90)
 		(unit 1)
@@
 		(dnp no)
 		(fields_autoplaced yes)
-		(property "Reference" "SW1"
-			(at 168.91 99.0599 90)
+		(property "Reference" "JP6"
+			(at 165.1 99.0599 90)
 			(effects
 				(font
@@
 		)
 		(property "Value" "MASTER"
-			(at 168.91 101.5999 90)
+			(at 165.1 101.5999 90)
 			(effects
 				(font
@@
 			)
 		)
-		(property "Footprint" ""
+		(property "Footprint" "Jumper:SolderJumper-2_P1.3mm_Bridged_RoundedPad1.0x1.5mm"
 			(at 163.83 100.33 0)
 			(effects
@@
 		)
 		(property "Datasheet" "~"
-			(at 171.45 100.33 0)
-			(effects
-				(font
-					(size 1.27 1.27)
-				)
-				(hide yes)
-			)
-		)
-		(property "Description" "Switch, single pole double throw"
 			(at 163.83 100.33 0)
 			(effects
@@
 			)
 		)
-		(pin "3"
+		(property "Description" "Jumper, 2-pole, small symbol, bridged"
+			(at 163.83 100.33 0)
+			(effects
+				(font
+					(size 1.27 1.27)
+				)
+				(hide yes)
+			)
+		)
+		(pin "2"
 		)
 		(pin "1"
 		)
-		(pin "2"
-		)
 		(instances
-			(project "LINBoard-HW"
+			(project ""
 				(path "/27863e5d-8a22-474c-850d-36d8970b0f4a/ff1b1819-f305-4259-a9f0-6b6ad7c927fb"
-					(reference "SW1")
+					(reference "JP6")
 					(unit 1)
 				)
@@
 			)
 		)
-		(property "Footprint" "Resistor_SMD:R_0603_1608Metric"
+		(property "Footprint" "Resistor_SMD:R_0402_1005Metric"
 			(at 111.76 92.71 0)
 			(effects
@@
 			)
 		)
-		(property "Footprint" "Capacitor_SMD:C_0603_1608Metric"
+		(property "Footprint" "Capacitor_SMD:C_0402_1005Metric"
 			(at 119.38 85.09 0)
 			(effects
@@
 			)
 		)
-		(property "Footprint" "Capacitor_SMD:C_0603_1608Metric"
+		(property "Footprint" "Capacitor_SMD:C_0402_1005Metric"
 			(at 157.48 113.03 0)
 			(effects
@@
 	(symbol
 		(lib_id "Device:R_Small_US")
-		(at 166.37 91.44 0)
+		(at 163.83 91.44 0)
 		(unit 1)
 		(exclude_from_sim no)
@@
 		(fields_autoplaced yes)
 		(property "Reference" "R1"
-			(at 168.91 90.1699 0)
+			(at 166.37 90.1699 0)
 			(effects
 				(font
@@
 		)
 		(property "Value" "1K"
-			(at 168.91 92.7099 0)
+			(at 166.37 92.7099 0)
 			(effects
 				(font
@@
 			)
 		)
-		(property "Footprint" "Resistor_SMD:R_0603_1608Metric"
-			(at 166.37 91.44 0)
+		(property "Footprint" "Resistor_SMD:R_0402_1005Metric"
+			(at 163.83 91.44 0)
 			(effects
 				(font
@@
 		)
 		(property "Datasheet" "~"
-			(at 166.37 91.44 0)
+			(at 163.83 91.44 0)
 			(effects
 				(font
@@
 		)
 		(property "Description" "Resistor, small US symbol"
-			(at 166.37 91.44 0)
+			(at 163.83 91.44 0)
 			(effects
 				(font
@@
 	)
 	(symbol
+		(lib_id "power:+3.3V")
+		(at 111.76 87.63 0)
+		(unit 1)
+		(exclude_from_sim no)
+		(in_bom yes)
+		(on_board yes)
+		(dnp no)
+		(fields_autoplaced yes)
+		(property "Reference" "#PWR06"
+			(at 111.76 91.44 0)
+			(effects
+				(font
+					(size 1.27 1.27)
+				)
+				(hide yes)
+			)
+		)
+		(property "Value" "+3.3V"
+			(at 111.76 82.55 0)
+			(effects
+				(font
+					(size 1.27 1.27)
+				)
+			)
+		)
+		(property "Footprint" ""
+			(at 111.76 87.63 0)
+			(effects
+				(font
+					(size 1.27 1.27)
+				)
+				(hide yes)
+			)
+		)
+		(property "Datasheet" ""
+			(at 111.76 87.63 0)
+			(effects
+				(font
+					(size 1.27 1.27)
+				)
+				(hide yes)
+			)
+		)
+		(property "Description" "Power symbol creates a global label with name \"+3.3V\""
+			(at 111.76 87.63 0)
+			(effects
+				(font
+					(size 1.27 1.27)
+				)
+				(hide yes)
+			)
+		)
+		(pin "1"
+		)
+		(instances
+			(project ""
+				(path "/27863e5d-8a22-474c-850d-36d8970b0f4a/ff1b1819-f305-4259-a9f0-6b6ad7c927fb"
+					(reference "#PWR06")
+					(unit 1)
+				)
+			)
+		)
+	)
+	(symbol
 		(lib_id "dk_TVS-Diodes:PESD1LIN")
 		(at 176.53 114.3 270)
@@
 			)
 		)
-		(property "Footprint" ""
+		(property "Footprint" "Diode_SMD:D_SOD-323"
 			(at 176.53 114.3 0)
 			(effects
@@
 	(symbol
 		(lib_id "Device:D_Schottky_Small_Filled")
-		(at 166.37 83.82 90)
+		(at 163.83 83.82 90)
 		(unit 1)
 		(exclude_from_sim no)
@@
 		(fields_autoplaced yes)
 		(property "Reference" "D2"
-			(at 168.91 82.8039 90)
+			(at 166.37 82.8039 90)
 			(effects
 				(font
@@
 			)
 		)
-		(property "Value" "D_Schottky_Small_Filled"
-			(at 168.91 85.3439 90)
+		(property "Value" "Schottky"
+			(at 166.37 85.3439 90)
 			(effects
 				(font
@@
 			)
 		)
-		(property "Footprint" ""
-			(at 166.37 83.82 90)
+		(property "Footprint" "Diode_SMD:D_SOD-123"
+			(at 163.83 83.82 90)
 			(effects
 				(font
@@
 		)
 		(property "Datasheet" "~"
-			(at 166.37 83.82 90)
+			(at 163.83 83.82 90)
 			(effects
 				(font
@@
 		)
 		(property "Description" "Schottky diode, small symbol, filled shape"
-			(at 166.37 83.82 0)
-			(effects
-				(font
+			(at 163.83 83.82 0)
+			(effects
+				(font

Commit message: doing some layout
Parts:
- C1, C2: footprint Capacitor_SMD:C_0402_1005Metric -> Capacitor_SMD:C_0805_2012Metric
- R1, R2: footprint Resistor_SMD:R_0402_1005Metric -> Resistor_SMD:R_0805_2012Metric
Changed lines of the file:
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@@
 			)
 		)
-		(property "Footprint" "Resistor_SMD:R_0402_1005Metric"
+		(property "Footprint" "Resistor_SMD:R_0805_2012Metric"
 			(at 111.76 92.71 0)
 			(effects
@@
 			)
 		)
-		(property "Footprint" "Capacitor_SMD:C_0402_1005Metric"
+		(property "Footprint" "Capacitor_SMD:C_0805_2012Metric"
 			(at 119.38 85.09 0)
 			(effects
@@
 			)
 		)
-		(property "Footprint" "Capacitor_SMD:C_0402_1005Metric"
+		(property "Footprint" "Capacitor_SMD:C_0805_2012Metric"
 			(at 157.48 113.03 0)
 			(effects
@@
 			)
 		)
-		(property "Footprint" "Resistor_SMD:R_0402_1005Metric"
+		(property "Footprint" "Resistor_SMD:R_0805_2012Metric"
 			(at 163.83 91.44 0)
 			(effects

Commit message: routing first pass complete
Parts:
- removed JP6: MASTER, Jumper:SolderJumper-2_P1.3mm_Bridged_RoundedPad1.0x1.5mm, symbol Jumper:Jumper_2_Small_Bridged
- added SW3: MASTER, SlideSwitch:CJS-1200TB, symbol Switch:SW_SPDT
Connections:
- net LIN: now also SW3.2 (B)
- net at R1.2: now also SW3.1 (A)
- no-connect marks 0 -> 1
Changed lines of the file:
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@@
 	)
 	(junction
-		(at 163.83 106.68)
+		(at 166.37 106.68)
 		(diameter 0)
 		(color 0 0 0 0)
@@
 		(color 0 0 0 0)
 	)
-	(wire
-		(pts
-			(xy 163.83 102.87) (xy 163.83 106.68)
-		)
-		(stroke
-			(width 0)
-			(type default)
-		)
+	(no_connect
+		(at 168.91 93.98)
 	)
 	(wire
@@
 	(wire
 		(pts
-			(xy 163.83 106.68) (xy 176.53 106.68)
-		)
-		(stroke
-			(width 0)
-			(type default)
-		)
-	)
-	(wire
-		(pts
 			(xy 130.81 76.2) (xy 130.81 77.47)
 		)
@@
 	(wire
 		(pts
+			(xy 166.37 106.68) (xy 176.53 106.68)
+		)
+		(stroke
+			(width 0)
+			(type default)
+		)
+	)
+	(wire
+		(pts
+			(xy 166.37 104.14) (xy 166.37 106.68)
+		)
+		(stroke
+			(width 0)
+			(type default)
+		)
+	)
+	(wire
+		(pts
 			(xy 106.68 101.6) (xy 118.11 101.6)
 		)
@@
 	(wire
 		(pts
-			(xy 163.83 93.98) (xy 163.83 97.79)
-		)
-		(stroke
-			(width 0)
-			(type default)
-		)
-	)
-	(wire
-		(pts
 			(xy 111.76 99.06) (xy 118.11 99.06)
 		)
@@
 	(wire
 		(pts
-			(xy 157.48 106.68) (xy 163.83 106.68)
+			(xy 157.48 106.68) (xy 166.37 106.68)
 		)
 		(stroke
@@
 			)
 			(justify right)
-		)
-	)
-	(symbol
-		(lib_id "Jumper:Jumper_2_Small_Bridged")
-		(at 163.83 100.33 90)
-		(unit 1)
-		(exclude_from_sim no)
-		(in_bom yes)
-		(on_board yes)
-		(dnp no)
-		(fields_autoplaced yes)
-		(property "Reference" "JP6"
-			(at 165.1 99.0599 90)
-			(effects
-				(font
-					(size 1.27 1.27)
-				)
-				(justify right)
-			)
-		)
-		(property "Value" "MASTER"
-			(at 165.1 101.5999 90)
-			(effects
-				(font
-					(size 1.27 1.27)
-				)
-				(justify right)
-			)
-		)
-		(property "Footprint" "Jumper:SolderJumper-2_P1.3mm_Bridged_RoundedPad1.0x1.5mm"
-			(at 163.83 100.33 0)
-			(effects
-				(font
-					(size 1.27 1.27)
-				)
-				(hide yes)
-			)
-		)
-		(property "Datasheet" "~"
-			(at 163.83 100.33 0)
-			(effects
-				(font
-					(size 1.27 1.27)
-				)
-				(hide yes)
-			)
-		)
-		(property "Description" "Jumper, 2-pole, small symbol, bridged"
-			(at 163.83 100.33 0)
-			(effects
-				(font
-					(size 1.27 1.27)
-				)
-				(hide yes)
-			)
-		)
-		(pin "2"
-		)
-		(pin "1"
-		)
-		(instances
-			(project ""
-				(path "/27863e5d-8a22-474c-850d-36d8970b0f4a/ff1b1819-f305-4259-a9f0-6b6ad7c927fb"
-					(reference "JP6")
-					(unit 1)
-				)
-			)
 		)
 	)
@@
 		(on_board yes)
 		(dnp no)
-		(fields_autoplaced yes)
 		(property "Reference" "R1"
-			(at 166.37 90.1699 0)
+			(at 159.258 90.424 0)
 			(effects
 				(font
@@
 		)
 		(property "Value" "1K"
-			(at 166.37 92.7099 0)
+			(at 159.258 92.964 0)
 			(effects
 				(font
@@
 					(unit 1)
 				)
+			)
+		)
+	)
+	(symbol
+		(lib_id "Switch:SW_SPDT")
+		(at 166.37 99.06 90)
+		(unit 1)
+		(exclude_from_sim no)
+		(in_bom yes)
+		(on_board yes)
+		(dnp no)
+		(fields_autoplaced yes)
+		(property "Reference" "SW3"
+			(at 171.45 97.7899 90)
+			(effects
+				(font
+					(size 1.27 1.27)
+				)
+				(justify right)
+			)
+		)
+		(property "Value" "MASTER"
+			(at 171.45 100.3299 90)
+			(effects
+				(font
+					(size 1.27 1.27)
+				)
+				(justify right)
+			)
+		)
+		(property "Footprint" "SlideSwitch:CJS-1200TB"
+			(at 166.37 99.06 0)
+			(effects
+				(font
+					(size 1.27 1.27)
+				)
+				(hide yes)
+			)
+		)
+		(property "Datasheet" "~"
+			(at 173.99 99.06 0)
+			(effects
+				(font
+					(size 1.27 1.27)
+				)
+				(hide yes)
+			)
+		)
+		(property "Description" "Switch, single pole double throw"
+			(at 166.37 99.06 0)
+			(effects
+				(font
+					(size 1.27 1.27)
+				)
+				(hide yes)
+			)
+		)
+		(pin "2"
+		)
+		(pin "1"
+		)
+		(pin "3"
+		)
+		(instances
+			(project "LINBoard-HW"
+				(path "/27863e5d-8a22-474c-850d-36d8970b0f4a/ff1b1819-f305-4259-a9f0-6b6ad7c927fb"
+					(reference "SW3")
+					(unit 1)
+				)

Commit message: add fab outputs
Parts:
- C2: LCSC Part (none) -> C49678
- D1: LCSC Part (none) -> C2858716
- D2: LCSC Part (none) -> C179426
- R1: LCSC Part (none) -> C17513
- R2: LCSC Part (none) -> C17526
- SW3: now left out of the parts list
- U2: LCSC Part (none) -> C194435
Changed lines of the file:
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@@
+			)
+		)
+		(property "LCSC Part" "C194435"
+			(at 130.81 104.14 0)
+			(effects
+				(font
+					(size 1.27 1.27)
+				)
+				(hide yes)
 			)
 		)
@@
 			)
 		)
+		(property "LCSC Part" "C17526"
+			(at 111.76 92.71 0)
+			(effects
+				(font
+					(size 1.27 1.27)
+				)
+				(hide yes)
+			)
+		)
 		(pin "1"
 		)
@@
 			)
 		)
+		(property "LCSC Part" "C49678"
+			(at 119.38 85.09 0)
+			(effects
+				(font
+					(size 1.27 1.27)
+				)
+				(hide yes)
+			)
+		)
 		(pin "1"
 		)
@@
 			)
 		)
+		(property "LCSC Part" ""
+			(at 157.48 113.03 0)
+			(effects
+				(font
+					(size 1.27 1.27)
+				)
+				(hide yes)
+			)
+		)
 		(pin "1"
 		)
@@
 			)
 		)
+		(property "LCSC Part" "C17513"
+			(at 163.83 91.44 0)
+			(effects
+				(font
+					(size 1.27 1.27)
+				)
+				(hide yes)
+			)
+		)
 		(pin "1"
 		)
@@
 			)
 		)
+		(property "LCSC Part" "C2858716"
+			(at 176.53 114.3 90)
+			(effects
+				(font
+					(size 1.27 1.27)
+				)
+				(hide yes)
+			)
+		)
 		(pin "1"
 		)
@@
 		(unit 1)
 		(exclude_from_sim no)
-		(in_bom yes)
+		(in_bom no)
 		(on_board yes)
 		(dnp no)
@@
 			)
 		)
+		(property "LCSC Part" ""
+			(at 166.37 99.06 90)
+			(effects
+				(font
+					(size 1.27 1.27)
+				)
+				(hide yes)
+			)
+		)
 		(pin "2"
 		)
@@
 			(effects
 				(font
+					(size 1.27 1.27)
+				)
+				(hide yes)
+			)
+		)
+		(property "LCSC Part" "C179426"
+			(at 163.83 83.82 90)
+			(effects
+				(font

Commit message: change pinout, export
Parts:
- C1: LCSC Part (none) -> C576920
Changed lines of the file:
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@@
 			)
 		)
-		(property "LCSC Part" ""
+		(property "LCSC Part" "C576920"
 			(at 157.48 113.03 0)
 			(effects
